File: sv16_board_placed_native.kicad_pcb (KiCad board)
At the start: 4 copper layers, 122 x 122.8 mm, 141 parts, among them J1 JTAG, J10 CONSOLE, J2 JTAG-1.27, J3 EXP-A, J4 EXP-B, J5 EXP-C, J6 MOTOR, J7 SPARE (not fitted), J8 USB-C, J9 7-12 V, Q1 2N7002, Q2 BC817, Q4 BC807, SW1 RESET, SW2 RECONFIG, U1 LFE5U-12F-6TG144C, U2 W25Q64JVSSIQ, U3 W25Q64JVSSIQ, U4 CH340G, U5 AP62300TWU-7, U6 MP1584EN, U7 LP5907MFX-2.5, U8 USBLC6-2SC6, Y1 25 MHz ACTIVE XO (4-pin), Y2 12 MHz (CH340G clock)

Commit message: Y1: record ECS-2333-250-BN-TR 25MHz 3.3V XO part value (verified clock path, no placement/net changes)
Co-authored-by: arena-agent <297053741+arena-agent@users.noreply.github.com>
Parts:
- Y1: value 25 MHz ACTIVE XO (4-pin) -> ECS-2333-250-BN-TR 25MHz 3.3V XO
Changed lines of the file:
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@@
 			)
 		)
-		(property "Value" "25 MHz ACTIVE XO (4-pin)"
+		(property "Value" "ECS-2333-250-BN-TR 25MHz 3.3V XO"
 			(at 0 2.45 0)
 			(layer "F.Fab")
